Commit message: feat: add Lula kinematic solver support
- Integrate Lula kinematic solver functionality  
- Enable IK solving using Lula configuration files  
- Connect solver with OpenArm control pipeline

File: isaacsim.openarm_UI/openarm_UI/assets/openarm_bimanual.urdf (robot description, URDF)
Before this commit: robot openarm, 26 links, 25 joints
Joints:
- joint openarm_right_joint5: axis 1 0 0 -> 0 0 1
